Commit message: training results added, still no success

File: rl_walker_description/urdf/bot.xacro (robot description, xacro)
@@ -6,5 +6,5 @@
     <origin xyz="0.0 0.0 0.0" rpy="0 0 0" />
     <mass value="0.3" />
-    <inertia ixx="0.1" ixy="0.1" ixz="0.1" iyy="0.1" iyz="0.1" izz="0.1"/>
+    <inertia ixx="0.000000001" ixy="0.000000001" ixz="0.000000001" iyy="0.000000001" iyz="0.000000001" izz="0.000000001"/>
 </inertial>
 <visual>
@@ -24,5 +24,5 @@
 <inertial>
     <origin xyz="0.0 0.0 0.5" rpy="0 0 0" />
-    <mass value="4.0" />
+    <mass value="3.0" />
     <inertia ixx="0.42841" ixy="-2.3739" ixz="0.00227" iyy="0.43178" iyz="1.46390" izz="0.08742"/>
 </inertial>
@@ -55,5 +55,5 @@
     <child link="bum_zl" />
     <axis xyz="0 0 1" />
-    <limit lower="-0.345" upper="0.345" effort="1000" velocity="3"/>
+    <limit lower="-0.345" upper="0.345" effort="20" velocity="3"/>
     <!-- dynamics damping="5" friction="0.0"/ -->
 </joint>
@@ -62,5 +62,5 @@
     <origin xyz="0.0 0.0 -0.19" rpy="0 0 0" />
     <mass value="0.3" />
-    <inertia ixx="0.1" ixy="0.1" ixz="0.1" iyy="0.1" iyz="0.1" izz="0.1"/>
+    <inertia ixx="0.000000001" ixy="0.000000001" ixz="0.000000001" iyy="0.000000001" iyz="0.000000001" izz="0.000000001"/>
 </inertial>
 <visual>
@@ -83,5 +83,5 @@
     <child link="bum_xl" />
     <axis xyz="1 0 0" />
-    <limit lower="-0.345" upper="1" effort="1000" velocity="3"/>
+    <limit lower="-0.345" upper="1" effort="20" velocity="3"/>
     <!-- dynamics damping="5" friction="0.0"/ -->
 </joint>
@@ -90,5 +90,5 @@
     <origin xyz="0.0 0.0 -0.19" rpy="0 0 0" />
     <mass value="0.3" />
-    <inertia ixx="0.1" ixy="0.1" ixz="0.1" iyy="0.1" iyz="0.1" izz="0.1"/>
+    <inertia ixx="0.000000001" ixy="0.000000001" ixz="0.000000001" iyy="0.000000001" iyz="0.000000001" izz="0.000000001"/>
 </inertial>
 <visual>
@@ -112,5 +112,5 @@
     <child link="left_hip" />
     <axis xyz="0 1 0" />
-    <limit lower="0" upper="1" effort="1000" velocity="3"/>
+    <limit lower="0" upper="1" effort="20" velocity="3"/>
     <!-- dynamics damping="5" friction="0.0"/ -->
 </joint>
@@ -140,5 +140,5 @@
     <child link="left_shin" />
     <axis xyz="0 1 0" />
-    <limit lower="-1.3" upper="0" effort="1000" velocity="3"/>
+    <limit lower="-1.3" upper="0" effort="20" velocity="3"/>
     <!-- dynamics damping="5" friction="0.0"/ -->
 </joint>
@@ -169,5 +169,5 @@
     <child link="left_ankle" />
     <axis xyz="0 1 0" />
-    <limit lower="-1.3" upper="0.3" effort="1000" velocity="3"/>
+    <limit lower="-1.3" upper="0.3" effort="20" velocity="3"/>
 </joint>
 <link name="left_ankle">
@@ -196,10 +196,10 @@
     <child link="left_foot" />
     <axis xyz="0 1 0" />
-    <limit lower="-0.4" upper="0.7" effort="1000" velocity="3"/>
+    <limit lower="-0.4" upper="0.7" effort="20" velocity="3"/>
 </joint>
 <link name="left_foot">
 <inertial>
     <origin xyz="0.0 0.0 0" rpy="0 0 0" />
-    <mass value="0.5" />
+    <mass value="1.5" />
     <inertia ixx="0.10917" ixy="1.3005" ixz="-0.01020" iyy="0.15687" iyz="3.44815" izz="0.1"/>
 </inertial>
@@ -223,5 +223,5 @@
     <child link="left_leg_contact_sensor" />
     <axis xyz="0 1 0" />
-    <!-- <limit lower="-0.4" upper="0.7" effort="1000" velocity="3"/> -->
+    <!-- <limit lower="-0.4" upper="0.7" effort="20" velocity="3"/> -->
     <!-- dynamics damping="5" friction="0.0"/ -->
 </joint>
@@ -262,5 +262,5 @@
     <child link="bum_zr" />
     <axis xyz="0 0 1" />
-    <limit lower="-0.345" upper="0.345" effort="1000" velocity="3"/>
+    <limit lower="-0.345" upper="0.345" effort="20" velocity="3"/>
     <!-- dynamics damping="5" friction="0.0"/ -->
 </joint>
@@ -269,5 +269,5 @@
     <origin xyz="0.0 0.0 -0.19" rpy="0 0 0" />
     <mass value="0.3" />
-    <inertia ixx="0.1" ixy="0.1" ixz="0.1" iyy="0.1" iyz="0.1" izz="0.1"/>
+    <inertia ixx="0.000000001" ixy="0.000000001" ixz="0.000000001" iyy="0.000000001" iyz="0.000000001" izz="0.000000001"/>
 </inertial>
 <visual>
@@ -290,5 +290,5 @@
     <child link="bum_xr" />
     <axis xyz="1 0 0" />
-    <limit lower="-1" upper="0.345" effort="1000" velocity="3"/>
+    <limit lower="-1" upper="0.345" effort="20" velocity="3"/>
     <!-- dynamics damping="5" friction="0.0"/ -->
 </joint>
@@ -297,5 +297,5 @@
     <origin xyz="0.0 0.0 -0.19" rpy="0 0 0" />
     <mass value="0.3" />
-    <inertia ixx="0.1" ixy="0.1" ixz="0.1" iyy="0.1" iyz="0.1" izz="0.1"/>
+    <inertia ixx="0.000000001" ixy="0.000000001" ixz="0.000000001" iyy="0.000000001" iyz="0.000000001" izz="0.000000001"/>
 </inertial>
 <visual>
@@ -318,5 +318,5 @@
     <child link="right_hip" />
     <axis xyz="0 1 0" />
-    <limit lower="0" upper="1" effort="1000" velocity="3"/>
+    <limit lower="0" upper="1" effort="20" velocity="3"/>
     <!-- dynamics damping="5" friction="0.0"/ -->
 </joint>
@@ -346,5 +346,5 @@
     <child link="right_shin" />
     <axis xyz="0 1 0" />
-    <limit lower="-1.3" upper="0" effort="1000" velocity="3"/>
+    <limit lower="-1.3" upper="0" effort="20" velocity="3"/>
     <!-- dynamics damping="5" friction="0.0"/ -->
 </joint>
@@ -374,5 +374,5 @@
     <child link="right_ankle" />
     <axis xyz="0 1 0" />
-    <limit lower="-1.3" upper="0.3" effort="1000" velocity="3"/>
+    <limit lower="-1.3" upper="0.3" effort="20" velocity="3"/>
 </joint>
 <link name="right_ankle">
@@ -401,5 +401,5 @@
     <child link="right_foot" />
     <axis xyz="0 1 0" />
-    <limit lower="-0.4" upper="0.7" effort="1000" velocity="3"/>
+    <limit lower="-0.4" upper="0.7" effort="20" velocity="3"/>
     <!-- dynamics damping="5" friction="0.0"/ -->
 </joint>
@@ -407,5 +407,5 @@
 <inertial>
     <origin xyz="0.0 0.0 0.0" rpy="0 0 0" />
-    <mass value="0.5" />
+    <mass value="1.5" />
     <inertia ixx="0.119924" ixy="-0.0003874" ixz="-0.0010433" iyy="0.166674" iyz="5.8010177" izz="0.1314669"/>
 </inertial>
@@ -429,5 +429,5 @@
     <child link="right_leg_contact_sensor" />
     <axis xyz="0 1 0" />
-    <!-- <limit lower="-" upper="0.7" effort="1000" velocity="3"/> -->
+    <!-- <limit lower="-" upper="0.7" effort="20" velocity="3"/> -->
     <!-- dynamics damping="5" friction="0.0"/ -->
 </joint>
@@ -462,5 +462,5 @@
      ######################### right hand ########################
      ########################################################## -->
-<joint
+<!-- <joint
     name="shoulder_zrj" type="revolute">
     <origin xyz="0 -0.3 0.87" rpy="0 0 0" />
@@ -468,12 +468,11 @@
     <child link="shoulder_zr" />
     <axis xyz="0 0 1" />
-    <limit lower="-0.345" upper="1.65" effort="1000" velocity="3"/>
-    <!-- dynamics damping="5" friction="0.0"/ -->
+    <limit lower="-0.345" upper="1.65" effort="20" velocity="3"/>
 </joint>
 <link name="shoulder_zr">
 <inertial>
     <origin xyz="0.0 0.0 0.0" rpy="0 0 0" />
-    <mass value="0.3" />
-    <inertia ixx="0.1" ixy="0.1" ixz="0.1" iyy="0.1" iyz="0.1" izz="0.1"/>
+    <mass value="0.1" />
+    <inertia ixx="0.000000001" ixy="0.000000001" ixz="0.000000001" iyy="0.000000001" iyz="0.000000001" izz="0.000000001"/>
 </inertial>
 <visual>
@@ -496,12 +495,11 @@
     <child link="shoulder_xr" />
     <axis xyz="1 0 0" />
-    <limit lower="-0.1" upper="1.6" effort="1000" velocity="3"/>
-    <!-- dynamics damping="5" friction="0.0"/ -->
+    <limit lower="-0.1" upper="1.6" effort="20" velocity="3"/>
 </joint>
 <link name="shoulder_xr">
 <inertial>
     <origin xyz="0.0 0.0 0.0" rpy="0 0 0" />
-    <mass value="0.3" />
-    <inertia ixx="0.1" ixy="0.1" ixz="0.1" iyy="0.1" iyz="0.1" izz="0.1"/>
+    <mass value="0.1" />
+    <inertia ixx="0.000000001" ixy="0.000000001" ixz="0.000000001" iyy="0.000000001" iyz="0.000000001" izz="0.000000001"/>
 </inertial>
 <visual>
@@ -524,11 +522,10 @@
     <child link="right_shoulder" />
     <axis xyz="0 1 0" />
-    <limit lower="0" upper="3" effort="1000" velocity="3"/>
-    <!-- dynamics damping="5" friction="0.0"/ -->
+    <limit lower="0" upper="3" effort="20" velocity="3"/>
 </joint>
 <link name="right_shoulder">
 <inertial>
     <origin xyz="0.0 0.0 0.0" rpy="0 0 0" />
-    <mass value="0.3" />
+    <mass value="0.1" />
     <inertia ixx="0.030306" ixy="1.072426" ixz="-0.00014" iyy="0.123799" iyz="-3.24634" izz="0.10389"/>
 </inertial>
@@ -552,11 +549,10 @@
     <child link="right_forearm" />
     <axis xyz="1 0 0" />
-    <limit lower="-1.6" upper="0" effort="1000" velocity="3"/>
-    <!-- dynamics damping="5" friction="0.0"/ -->
+    <limit lower="-1.6" upper="0" effort="20" velocity="3"/>
 </joint>
 <link name="right_forearm">
 <inertial>
     <origin xyz="0.0 0.0 0.0" rpy="0 0 0" />
-    <mass value="0.3" />
+    <mass value="0.1" />
     <inertia ixx="0.37633" ixy="-5.2759" ixz="-8.13739" iyy="0.382769" iyz="-0.00136" izz="0.03977"/>
 </inertial>
@@ -573,9 +569,9 @@
     </geometry>
 </collision>
-</link>
+</link> -->
 <!-- ##########################################################
      ######################### right left ########################
      ########################################################## -->
-<joint
+<!-- <joint
     name="shoulder_zlj" type="revolute">
     <origin xyz="0 0.3 0.87" rpy="0 0 3.142" />
@@ -583,12 +579,11 @@
     <child link="shoulder_zl" />
     <axis xyz="0 0 1" />
-    <limit lower="-1.65" upper="0.1" effort="1000" velocity="3"/>
-    <!-- dynamics damping="5" friction="0.0"/ -->
+    <limit lower="-1.65" upper="0.1" effort="20" velocity="3"/>
 </joint>
 <link name="shoulder_zl">
 <inertial>
     <origin xyz="0.0 0.0 0.0" rpy="0 0 0" />
-    <mass value="0.3" />
-    <inertia ixx="0.1" ixy="0.1" ixz="0.1" iyy="0.1" iyz="0.1" izz="0.1"/>
+    <mass value="0.1" />
+    <inertia ixx="0.000000001" ixy="0.000000001" ixz="0.000000001" iyy="0.000000001" iyz="0.000000001" izz="0.000000001"/>
 </inertial>
 <visual>
@@ -611,12 +606,11 @@
     <child link="shoulder_xl" />
     <axis xyz="1 0 0" />
-    <limit lower="-0.1" upper="1.6" effort="1000" velocity="3"/>
-    <!-- dynamics damping="5" friction="0.0"/ -->
+    <limit lower="-0.1" upper="1.6" effort="20" velocity="3"/>
 </joint>
 <link name="shoulder_xl">
 <inertial>
     <origin xyz="0.0 0.0 0.0" rpy="0 0 0" />
-    <mass value="0.3" />
-    <inertia ixx="0.1" ixy="0.1" ixz="0.1" iyy="0.1" iyz="0.1" izz="0.1"/>
+    <mass value="0.1" />
+    <inertia ixx="0.000000001" ixy="0.000000001" ixz="0.000000001" iyy="0.000000001" iyz="0.000000001" izz="0.000000001"/>
 </inertial>
 <visual>
@@ -639,11 +633,10 @@
     <child link="left_shoulder" />
     <axis xyz="0 1 0" />
-    <limit lower="-3" upper="0" effort="1000" velocity="3"/>
-    <!-- dynamics damping="5" friction="0.0"/ -->
+    <limit lower="-3" upper="0" effort="20" velocity="3"/>
 </joint>
 <link name="left_shoulder">
 <inertial>
     <origin xyz="0.0 0.0 0.0" rpy="0 0 0" />
-    <mass value="0.3" />
+    <mass value="0.1" />
     <inertia ixx="0.030306" ixy="1.072426" ixz="-0.00014" iyy="0.123799" iyz="-3.24634" izz="0.10389"/>
 </inertial>
@@ -667,11 +660,10 @@
     <child link="left_forearm" />
     <axis xyz="1 0 0" />
-    <limit lower="-1.6" upper="0" effort="1000" velocity="3"/>
-    <!-- dynamics damping="5" friction="0.0"/ -->
+    <limit lower="-1.6" upper="0" effort="20" velocity="3"/>
 </joint>
 <link name="left_forearm">
 <inertial>
     <origin xyz="0.0 0.0 0.0" rpy="0 0 0" />
-    <mass value="0.3" />
+    <mass value="0.1" />
     <inertia ixx="0.37633" ixy="-5.2759" ixz="-8.13739" iyy="0.382769" iyz="-0.00136" izz="0.03977"/>
 </inertial>
@@ -688,4 +680,4 @@
     </geometry>
 </collision>
-</link>
+</link> -->
 </robot>
